File: sensors/temperature-humidity/DHT22/battery-powered/kicad/wiring/wiring.kicad_sch (KiCad schematic)
At the start: 1 part

Commit message: feat: adding libraries to kikad
Parts:
- added TH?: DHT22_Temperature_Humidity, symbol sensors:DHT22_Temperature_Humidity
- added U?: nRF24L01+, MODULE, symbol nRF24L01+:nRF24L01+
Changed lines of the file:
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@@
 (kicad_sch (version 20211123) (generator eeschema)
   (paper "A4")
+  (symbol (lib_id "sensors:DHT22_Temperature_Humidity") (at 165.1 63.5 0) (unit 1)
+    (in_bom yes) (on_board yes) (fields_autoplaced)
+    (property "Reference" "TH?" (id 0) (at 172.72 48.895 0)
+      (effects (font (size 1.524 1.524)) (justify left))
+    )
+    (property "Value" "DHT22_Temperature_Humidity" (id 1) (at 172.72 52.705 0)
+      (effects (font (size 1.524 1.524)) (justify left))
+    )
+    (property "Footprint" "" (id 2) (at 165.1 63.5 0)
+      (effects (font (size 1.524 1.524)))
+    )
+    (property "Datasheet" "" (id 3) (at 165.1 63.5 0)
+      (effects (font (size 1.524 1.524)))
+    )
+    (pin "1")
+    (pin "2")
+    (pin "3")
+    (pin "4")
+  )
+  (symbol (lib_id "nRF24L01+:nRF24L01+") (at 167.64 93.98 0) (unit 1)
+    (in_bom yes) (on_board yes) (fields_autoplaced)
+    (property "Reference" "U?" (id 0) (at 167.64 80.01 0))
+    (property "Value" "nRF24L01+" (id 1) (at 167.64 82.55 0))
+    (property "Footprint" "MODULE" (id 2) (at 167.64 91.44 0)
+      (effects (font (size 1.27 1.27)) hide)
+    )
+    (property "Datasheet" "DOCUMENTATION" (id 3) (at 167.64 95.25 0)
+      (effects (font (size 1.27 1.27)) hide)
+    )
+    (pin "1")
+    (pin "2")
+    (pin "3")
+    (pin "4")
+    (pin "5")
+    (pin "6")
+    (pin "7")
+    (pin "8")
+  )
   (symbol (lib_id "arduino-pro-mini:arduino-pro-mini") (at 111.76 93.98 0) (unit 1)
     (in_bom yes) (on_board yes) (fields_autoplaced)
@@
   )
   (symbol_instances
+    (path "/0c4ec2cd-9fe3-4d02-bc3e-977e924425a1"
+      (reference "TH?") (unit 1) (value "DHT22_Temperature_Humidity") (footprint "")
+    )
+    (path "/223b12a9-5805-4cfc-9b47-dd8a97f2ab06"
+      (reference "U?") (unit 1) (value "nRF24L01+") (footprint "MODULE")
+    )
     (path "/573c3e86-fc56-40ad-bcb1-372b72b2c6fe"
       (reference "U?") (unit 1) (value "arduino-pro-mini") (footprint "")

Commit message: feat: adding schematics
Parts:
- added BT1, BT2: 1.5V, symbol Device:Battery_Cell
- TH1: renamed from TH?; footprint (none) -> Sensors:DHT22_Temperature_Humidity
- U2: renamed from U?; footprint MODULE -> RF_Module:nRF24L01_Breakout
- gave numbers to parts that had none: 1
Connections:
- net at TH1.1 (VDD): now also U1.21 (VCC), U2.2 (VCC), BT1.1 (+)
- net at TH1.2 (DATA): now also U1.6 (D3)
- net GND: now reaches TH1.4 (GND)
- net GND: now also U1.23 (GND), U2.1 (GND), BT2.2 (-)
- net at U2.3 (CE): now also U1.9 (D6)
- net at U2.4 (CSN): now also U1.10 (D7)
- net at U2.5 (SCK): now also U1.16 (D13)
- net at U2.6 (MOSI): now also U1.14 (D11)
- net at U2.7 (MISO): now also U1.15 (D12)
- net at U2.8 (IRQ): now also U1.5 (D2)
- new net: BT1.2 (-), BT2.1 (+)
Other:
- moved on the sheet: TH1, U1, U2

Commit message: feat: better wiring
Parts:
- removed BT2: 1.5V, symbol Device:Battery_Cell
- removed TH1: DHT22_Temperature_Humidity, Sensors:DHT22_Temperature_Humidity, symbol sensors:DHT22_Temperature_Humidity
- removed U1: arduino-pro-mini, symbol arduino-pro-mini:arduino-pro-mini
- added C1: 10µF, Capacitor_THT:C_Disc_D3.0mm_W1.6mm_P2.50mm, symbol Device:C
- added J1: Conn_01x01_Male, Connector_PinHeader_1.00mm:PinHeader_1x01_P1.00mm_Vertical, symbol Connector:Conn_01x01_Male
- added J2: BME280, Connector_PinHeader_2.54mm:PinHeader_1x06_P2.54mm_Vertical, symbol Connector:Conn_01x06_Male
- added U1: ARDUINO_PRO_MINI, ARDUINO_PRO_MINI:MODULE_ARDUINO_PRO_MINI, symbol ARDUINO_PRO_MINI:ARDUINO_PRO_MINI
- added U3: BME280, Package_LGA:Bosch_LGA-8_2.5x2.5mm_P0.65mm_ClockwisePinNumbering, symbol Sensor:BME280
- BT1: value 1.5V -> 2x1,5V; footprint (none) -> Battery:BatteryHolder_Keystone_2462_2xAA
Connections:
- net GND: now also BT1.2 (-), C1.2, J2.5 (Pin_5), U1.JP6_2 (GND_1), U3.1 (GND), U3.7 (GND)
- net at BT1.1 (+), U2.2 (VCC): now also C1.1, J1.1 (Pin_1), J2.6 (Pin_6), U1.JP6_4 (VCC_1), U3.8 (VDD)
- net at U2.3 (CE): now also U1.JP7_1 (D9)
- net at U2.4 (CSN): now also U1.JP6_12 (D10)
- net at U2.5 (SCK): now also U1.JP6_9 (SCK)
- net at U2.6 (MOSI): now also U1.JP6_11 (MOSI)
- net at U2.7 (MISO): now also U1.JP6_10 (MISO)
- net at U2.8 (IRQ): now also U1.JP7_8 (D2)
- new net: J2.2 (Pin_2), U3.2 (CSB)
- new net: J2.3 (Pin_3), U1.JP2_1 (A4), U3.3 (SDI)
- new net: J2.4 (Pin_4), U1.JP2_2 (A5), U3.4 (SCK)
- new net: J2.1 (Pin_1), U3.5 (SDO)
- new net: U1.JP1_5 (GND), U1.JP1_6 (GND)
